Commit message: 流程简化

File: src/aubo_ros2_driver/aubo_description/urdf/xacro/inc/aubo_ros2.xacro (robot description, xacro)
@@ -103,16 +103,16 @@
   <!-- TCP center of suction surface -->
   <link name="suction_tcp">
-    <!-- A tiny valid inertia prevents Gazebo's URDF->SDF conversion from
-         deleting this fixed child link before the suction plugin resolves it. -->
+    <!-- Keep the TCP as an independent Gazebo link for the suction plugin,
+         but avoid coupling a 50 g payload to a near-zero-mass body. -->
     <inertial>
       <origin xyz="0 0 0" rpy="0 0 0"/>
-      <mass value="0.0001"/>
+      <mass value="0.01"/>
       <inertia
-        ixx="0.00000001"
+        ixx="0.0000001667"
         ixy="0.0"
         ixz="0.0"
-        iyy="0.00000001"
+        iyy="0.0000001667"
         iyz="0.0"
-        izz="0.00000001"/>
+        izz="0.0000001667"/>
     </inertial>
   </link>

File: src/aubo_ros2_driver/aubo_description/urdf/xacro/inc/aubo_ros2_macro.xacro (robot description, xacro)
@@ -17,7 +17,9 @@
       <inertial>
         <origin xyz="0 0 0" rpy="0 0 0"/>
-        <mass value="0.0001"/>
-        <inertia ixx="0.00000001" ixy="0.0" ixz="0.0"
-                 iyy="0.00000001" iyz="0.0" izz="0.00000001"/>
+        <!-- Finite adapter inertia avoids an extreme mass ratio in the
+             preserved Gazebo fixed-joint chain. -->
+        <mass value="0.02"/>
+        <inertia ixx="0.0000003333" ixy="0.0" ixz="0.0"
+                 iyy="0.0000003333" iyz="0.0" izz="0.0000003333"/>
       </inertial>
     </link>
